Commit message: Fix bug

File: urdf/car.xacro (robot description, xacro)
@@ -2,9 +2,12 @@
 <robot xmlns:xacro="http://www.ros.org/wiki/xacro" name="car_simulation">
 <!--  -->
+  <!-- Import Rviz colors -->
+  <xacro:include filename="$(find car_simulation)/urdf/materials.xacro" />
+<!--  -->
   <xacro:property name="base_link_msh" value="package://car_simulation/meshes/base_link.STL" />
+  <xacro:property name="LF_wheel_msh" value="package://car_simulation/meshes/LF_wheel.STL" />
   <xacro:property name="LB_wheel_msh" value="package://car_simulation/meshes/LB_wheel.STL" />
-  <xacro:property name="LF_wheel_msh" value="package://car_simulation/meshes/LF_wheel.STL" />
+  <xacro:property name="RF_wheel_msh" value="package://car_simulation/meshes/RF_wheel.STL" />
   <xacro:property name="RB_wheel_msh" value="package://car_simulation/meshes/RB_wheel.STL" />
-  <xacro:property name="RF_wheel_msh" value="package://car_simulation/meshes/RF_wheel.STL" />
 <!--  -->
   <gazebo>
@@ -40,5 +43,5 @@
   </joint>
   <!--  -->
-  <xacro:macro name="links" params="part xyz_lnk ixx ixy ixz iyy iyz izz">
+  <xacro:macro name="links" params="part msh color mass xyz_lnk ixx ixy ixz iyy iyz izz">
     <gazebo reference="${part}">
       <material>Gazebo/Orange</material>
@@ -61,11 +64,7 @@
         <geometry>
           <mesh
-            filename="${${part}_msh}" />
+            filename="${msh}" />
         </geometry>
-        <material
-          name="">
-          <color
-            rgba="0.79216 0.81961 0.93333 1" />
-        </material>
+        <material name="${color}" />
       </visual>
       <collision>
@@ -75,5 +74,5 @@
         <geometry>
           <mesh
-            filename="${${part}_msh}" />
+            filename="${msh}" />
         </geometry>
       </collision>
@@ -81,7 +80,7 @@
   </xacro:macro>
   <!--  -->
-  <xacro:macro name="joints" params="part xyz_jnt x_axs">
+  <xacro:macro name="joints" params="part jnt xyz_jnt x_axs">
     <joint
-      name="${part}_jnt"
+      name="${jnt}"
       type="continuous">
       <origin
@@ -100,32 +99,31 @@
   </xacro:macro>
   <!--  -->
-  <xacro:links  part="base_link" mass="8"
+  <xacro:links  part="base_link" msh="${base_link_msh}" color="white" mass="8"
                 xyz_lnk="-0.00074513 -0.11739 0.055785"
                 ixx="0.55567" ixy="-0.00039063" ixz="-0.0032652"
                 iyy="0.57391" iyz="-0.019683" izz="0.61063"/>
   <!--  -->
-  <xacro:links  part="LF_wheel" mass="0.49554"
+  <xacro:links  part="LF_wheel" msh="${LF_wheel_msh}" color="orange" mass="0.49554"
                 xyz_lnk="-0.032026 -1.3878E-17 -5.5511E-17"
                 ixx="0.0018121" ixy="2.1263E-22" ixz="1.9263E-20"
                 iyy="0.00096656" iyz="5.0211E-21" izz="0.00096656"/>
-  <xacro:joints part="LF_wheel" xyz_jnt="-0.27192 0.1695 -0.1241" x_axs="1"/>
+  <xacro:joints part="LF_wheel" jnt="LF_wheel_jnt" xyz_jnt="-0.27192 0.1695 -0.1241" x_axs="1"/>
   <!--  -->
-  <xacro:links  part="LB_wheel" mass="0.49554"
+  <xacro:links  part="LB_wheel" msh="${LB_wheel_msh}" color="orange" mass="0.49554"
                 xyz_lnk="-0.032026 2.7756E-17 2.7756E-17"
                 ixx="0.0018121" ixy="2.1243E-20" ixz="3.9097E-21"
                 iyy="0.00096656" iyz="9.7862E-20" izz="0.00096656"/>
-  <xacro:joints part="LB_wheel" xyz_jnt="-0.27192 -0.2695 -0.1241" x_axs="1"/>
+  <xacro:joints part="LB_wheel" jnt="LB_wheel_jnt" xyz_jnt="-0.27192 -0.2695 -0.1241" x_axs="1"/>
   <!--  -->
-  <xacro:links part="RF_wheel" mass="0.49554"
+  <xacro:links part="RF_wheel" msh="${RF_wheel_msh}" color="orange" mass="0.49554"
                 xyz_lnk="0.032026 6.9389E-17 0"
-                xyz_jnt="0.27208 0.1695 -0.1241"
                 ixx="0.0018121" ixy="1.1755E-35" ixz="2.5636E-20"
                 iyy="0.00096656" iyz="3.8844E-35" izz="0.00096656"/>
-  <xacro:joints part="RF_wheel" xyz_jnt="0.27208 0.1695 -0.1241" x_axs="-1"/>
+  <xacro:joints part="RF_wheel" jnt="RF_wheel_jnt" xyz_jnt="0.27208 0.1695 -0.1241" x_axs="-1"/>
   <!--  -->
-  <xacro:links  part="RB_wheel" mass="0.49554"
-                xyz_jnt="0.27208 -0.2695 -0.1241"
+  <xacro:links  part="RB_wheel" msh="${RB_wheel_msh}" color="orange" mass="0.49554"
+                xyz_lnk="0.032026 6.9389E-17 0"
                 ixx="0.0018121" ixy="3.3987E-36" ixz="1.3212E-20"
                 iyy="0.00096656" iyz="-4.9432E-36" izz="0.00096656"/>
-  <xacro:joints part="RB_wheel" xyz_jnt="0.27208 -0.2695 -0.1241" x_axs="-1"/>
+  <xacro:joints part="RB_wheel" jnt="RB_wheel_jnt" xyz_jnt="0.27208 -0.2695 -0.1241" x_axs="-1"/>
 </robot>

Commit message: Update color display in gazebo world

File: urdf/car.xacro (robot description, xacro)
@@ -45,5 +45,10 @@
   <xacro:macro name="links" params="part msh color mass xyz_lnk ixx ixy ixz iyy iyz izz">
     <gazebo reference="${part}">
-      <material>Gazebo/Orange</material>
+      <xacro:if value="${color == 'white'}">
+        <material>Gazebo/White</material>
+      </xacro:if>
+      <xacro:if value="${color == 'orange'}">
+        <material>Gazebo/Orange</material>
+      </xacro:if>
     </gazebo>
     <link

Commit message: Update variables to control wheels

File: urdf/car.xacro (robot description, xacro)
@@ -1,8 +1,7 @@
 <?xml version="1.0" encoding="utf-8"?>
-<robot xmlns:xacro="http://www.ros.org/wiki/xacro" name="car_simulation">
-<!--  -->
+<robot xmlns:xacro="http://www.ros.org/wiki/xacro" name="car">
   <!-- Import Rviz colors -->
   <xacro:include filename="$(find car_simulation)/urdf/materials.xacro" />
-<!--  -->
+  <!-- Define the model path -->
   <xacro:property name="base_link_msh" value="package://car_simulation/meshes/base_link.STL" />
   <xacro:property name="LF_wheel_msh" value="package://car_simulation/meshes/LF_wheel.STL" />
@@ -10,37 +9,19 @@
   <xacro:property name="RF_wheel_msh" value="package://car_simulation/meshes/RF_wheel.STL" />
   <xacro:property name="RB_wheel_msh" value="package://car_simulation/meshes/RB_wheel.STL" />
-<!--  -->
+  <!-- Import gazebo plugins -->
   <gazebo>
     <plugin
       name="gazebo_ros_control"
       filename="libgazebo_ros_control.so">
-      <robotNamespace>/</robotNamespace>
+      <robotNamespace>/car</robotNamespace>
     </plugin>
   </gazebo>
-  <gazebo>
-    <plugin name="skid_steer_drive_controller" filename="libgazebo_ros_skid_steer_drive.so">
-      <legacyMode>false</legacyMode>
-      <alwaysOn>true</alwaysOn>
-      <updateRate>100.0</updateRate>
-      <robotNamespace>/</robotNamespace>
-      <leftFrontJoint>LF_wheel</leftFrontJoint>
-      <rightFrontJoint>RF_wheel</rightFrontJoint>
-      <leftRearJoint>LB_wheel</leftRearJoint>
-      <rightRearJoint>RB_wheel</rightRearJoint>
-      <wheelSeparation>0.4</wheelSeparation>
-      <wheelDiameter>0.215</wheelDiameter>
-      <robotBaseFrame>base_link</robotBaseFrame>
-      <torque>10</torque>
-      <topicName>cmd_vel</topicName>
-      <broadcastTF>false</broadcastTF>
-    </plugin>
-  </gazebo>
-  <!--  -->
+  <!-- Dummy link and joint used for baselink footprint -->
   <link name="dummy"></link>
-  <joint name="dummy_joint" type="fixed">
+  <joint name="dummy_jnt" type="fixed">
     <parent link="dummy"/>
     <child link="base_link"/>
   </joint>
-  <!--  -->
+  <!-- Macro for Links -->
   <xacro:macro name="links" params="part msh color mass xyz_lnk ixx ixy ixz iyy iyz izz">
     <gazebo reference="${part}">
@@ -84,5 +65,5 @@
     </link>
   </xacro:macro>
-  <!--  -->
+  <!-- Macro for Joints -->
   <xacro:macro name="joints" params="part jnt xyz_jnt x_axs">
     <joint
@@ -99,14 +80,29 @@
         xyz="${x_axs} 0 0" />
       <limit
-        effort="0"
-        velocity="35" />
+        effort="10"
+        velocity="100000" />
+      <dynamics
+        damping="0.8" />
     </joint>
   </xacro:macro>
-  <!--  -->
+  <!-- Macro for Wheel transmissions -->
+  <xacro:macro name="wheel_transmission" params="part jnt motor reduction">
+    <transmission name="${part}">
+      <type>transmission_interface/SimpleTransmission</type>
+      <joint name="${jnt}">
+        <hardwareInterface>hardware_interface/VelocityJointInterface</hardwareInterface>
+      </joint>
+      <actuator name="${motor}">
+        <hardwareInterface>hardware_interface/VelocityJointInterface</hardwareInterface>
+        <mechanicalReduction value="${reduction}" />
+      </actuator>
+    </transmission>
+  </xacro:macro>
+  <!-- base link setup -->
   <xacro:links  part="base_link" msh="${base_link_msh}" color="white" mass="8"
                 xyz_lnk="-0.00074513 -0.11739 0.055785"
                 ixx="0.55567" ixy="-0.00039063" ixz="-0.0032652"
                 iyy="0.57391" iyz="-0.019683" izz="0.61063"/>
-  <!--  -->
+  <!-- LF_wheel setup -->
   <xacro:links  part="LF_wheel" msh="${LF_wheel_msh}" color="orange" mass="0.49554"
                 xyz_lnk="-0.032026 -1.3878E-17 -5.5511E-17"
@@ -114,5 +110,6 @@
                 iyy="0.00096656" iyz="5.0211E-21" izz="0.00096656"/>
   <xacro:joints part="LF_wheel" jnt="LF_wheel_jnt" xyz_jnt="-0.27192 0.1695 -0.1241" x_axs="1"/>
-  <!--  -->
+  <xacro:wheel_transmission part="LF_wheel" jnt="LF_wheel_jnt" motor="LF_wheel_motor" reduction="1"/>
+  <!-- LB_wheel setup -->
   <xacro:links  part="LB_wheel" msh="${LB_wheel_msh}" color="orange" mass="0.49554"
                 xyz_lnk="-0.032026 2.7756E-17 2.7756E-17"
@@ -120,5 +117,6 @@
                 iyy="0.00096656" iyz="9.7862E-20" izz="0.00096656"/>
   <xacro:joints part="LB_wheel" jnt="LB_wheel_jnt" xyz_jnt="-0.27192 -0.2695 -0.1241" x_axs="1"/>
-  <!--  -->
+  <xacro:wheel_transmission part="LB_wheel" jnt="LB_wheel_jnt" motor="LB_wheel_motor" reduction="1"/>
+  <!-- RF_wheel setup -->
   <xacro:links part="RF_wheel" msh="${RF_wheel_msh}" color="orange" mass="0.49554"
                 xyz_lnk="0.032026 6.9389E-17 0"
@@ -126,5 +124,6 @@
                 iyy="0.00096656" iyz="3.8844E-35" izz="0.00096656"/>
   <xacro:joints part="RF_wheel" jnt="RF_wheel_jnt" xyz_jnt="0.27208 0.1695 -0.1241" x_axs="-1"/>
-  <!--  -->
+  <xacro:wheel_transmission part="RF_wheel" jnt="RF_wheel_jnt" motor="RF_wheel_motor" reduction="1"/>
+  <!-- RB_wheel setup -->
   <xacro:links  part="RB_wheel" msh="${RB_wheel_msh}" color="orange" mass="0.49554"
                 xyz_lnk="0.032026 6.9389E-17 0"
@@ -132,3 +131,4 @@
                 iyy="0.00096656" iyz="-4.9432E-36" izz="0.00096656"/>
   <xacro:joints part="RB_wheel" jnt="RB_wheel_jnt" xyz_jnt="0.27208 -0.2695 -0.1241" x_axs="-1"/>
+  <xacro:wheel_transmission part="RB_wheel" jnt="RB_wheel_jnt" motor="RB_wheel_motor" reduction="1"/>
 </robot>

Commit message: Import plugins seperately

File: urdf/car.xacro (robot description, xacro)
@@ -3,24 +3,45 @@
   <!-- Import Rviz colors -->
   <xacro:include filename="$(find car_simulation)/urdf/materials.xacro" />
+  <xacro:include filename="$(find car_simulation)/urdf/car.gazebo" />
   <!-- Define the model path -->
-  <xacro:property name="base_link_msh" value="package://car_simulation/meshes/base_link.STL" />
+  <xacro:property name="chassis_msh" value="package://car_simulation/meshes/chassis.STL" />
   <xacro:property name="LF_wheel_msh" value="package://car_simulation/meshes/LF_wheel.STL" />
   <xacro:property name="LB_wheel_msh" value="package://car_simulation/meshes/LB_wheel.STL" />
   <xacro:property name="RF_wheel_msh" value="package://car_simulation/meshes/RF_wheel.STL" />
   <xacro:property name="RB_wheel_msh" value="package://car_simulation/meshes/RB_wheel.STL" />
-  <!-- Import gazebo plugins -->
-  <gazebo>
-    <plugin
-      name="gazebo_ros_control"
-      filename="libgazebo_ros_control.so">
-      <robotNamespace>/car</robotNamespace>
-    </plugin>
-  </gazebo>
+  <xacro:property name="hokuyo_msh" value="package://car_simulation/meshes/hokuyo.dae"/>
   <!-- Dummy link and joint used for baselink footprint -->
-  <link name="dummy"></link>
-  <joint name="dummy_jnt" type="fixed">
-    <parent link="dummy"/>
-    <child link="base_link"/>
+  <link name="base_link"></link>
+  <joint name="base_jnt" type="fixed">
+    <parent link="base_link"/>
+    <child link="chassis"/>
   </joint>
+  <!-- Lidar Joint -->
+  <joint name="hokuyo_joint" type="fixed">
+    <axis xyz="0 1 0" />
+    <origin xyz="0 0 0.05" rpy="0 0 0"/>
+    <parent link="chassis"/>
+    <child link="hokuyo_link"/>
+  </joint>
+  <!-- Lidar Link -->
+  <link name="hokuyo_link">
+    <collision>
+      <origin xyz="0 0 0" rpy="0 0 0"/>
+      <geometry>
+        <box size="0.1 0.1 0.1"/>
+      </geometry>
+    </collision>
+    <visual>
+      <origin xyz="0 0 0" rpy="0 0 0"/>
+      <geometry>
+        <mesh filename="${hokuyo_msh}"/>
+      </geometry>
+    </visual>
+    <inertial>
+      <mass value="1E-5" />
+      <origin xyz="0 0 0" rpy="0 0 0"/>
+      <inertia ixx="1E-6" ixy="0" ixz="0" iyy="1E-6" iyz="0" izz="1E-6" />
+    </inertial>
+  </link>
   <!-- Macro for Links -->
   <xacro:macro name="links" params="part msh color mass xyz_lnk ixx ixy ixz iyy iyz izz">
@@ -74,5 +95,5 @@
         rpy="0 0 0" />
       <parent
-        link="base_link" />
+        link="chassis" />
       <child
         link="${part}"/>
@@ -100,5 +121,5 @@
   </xacro:macro>
   <!-- base link setup -->
-  <xacro:links  part="base_link" msh="${base_link_msh}" color="white" mass="8"
+  <xacro:links  part="chassis" msh="${chassis_msh}" color="white" mass="8"
                 xyz_lnk="-0.00074513 -0.11739 0.055785"
                 ixx="0.55567" ixy="-0.00039063" ixz="-0.0032652"

Commit message: Update Lidar scan

File: urdf/car.xacro (robot description, xacro)
@@ -29,5 +29,5 @@
       <origin xyz="0 0 0" rpy="0 0 0"/>
       <geometry>
-        <box size="0.1 0.1 0.1"/>
+        <mesh filename="${hokuyo_msh}"/>
       </geometry>
     </collision>

Commit message: Tidy up

File: urdf/car.xacro (robot description, xacro)
@@ -10,35 +10,35 @@
   <xacro:property name="RF_wheel_msh" value="package://car_simulation/meshes/RF_wheel.STL" />
   <xacro:property name="RB_wheel_msh" value="package://car_simulation/meshes/RB_wheel.STL" />
-  <xacro:property name="hokuyo_msh" value="package://car_simulation/meshes/hokuyo.dae"/>
+  <xacro:property name="hokuyo_msh" value="package://car_simulation/meshes/hokuyo.dae" />
   <!-- Dummy link and joint used for baselink footprint -->
   <link name="base_link"></link>
   <joint name="base_jnt" type="fixed">
-    <parent link="base_link"/>
-    <child link="chassis"/>
+    <parent link="base_link" />
+    <child link="chassis" />
   </joint>
   <!-- Lidar Joint -->
   <joint name="hokuyo_joint" type="fixed">
     <axis xyz="0 1 0" />
-    <origin xyz="0 0 0.05" rpy="0 0 0"/>
-    <parent link="chassis"/>
-    <child link="hokuyo_link"/>
+    <origin xyz="0 0 0.05" rpy="0 0 0" />
+    <parent link="chassis" />
+    <child link="hokuyo_link" />
   </joint>
   <!-- Lidar Link -->
   <link name="hokuyo_link">
     <collision>
-      <origin xyz="0 0 0" rpy="0 0 0"/>
+      <origin xyz="0 0 0" rpy="0 0 0" />
       <geometry>
-        <mesh filename="${hokuyo_msh}"/>
+        <mesh filename="${hokuyo_msh}" />
       </geometry>
     </collision>
     <visual>
-      <origin xyz="0 0 0" rpy="0 0 0"/>
+      <origin xyz="0 0 0" rpy="0 0 0" />
       <geometry>
-        <mesh filename="${hokuyo_msh}"/>
+        <mesh filename="${hokuyo_msh}" />
       </geometry>
     </visual>
     <inertial>
       <mass value="1E-5" />
-      <origin xyz="0 0 0" rpy="0 0 0"/>
+      <origin xyz="0 0 0" rpy="0 0 0" />
       <inertia ixx="1E-6" ixy="0" ixz="0" iyy="1E-6" iyz="0" izz="1E-6" />
     </inertial>
@@ -53,4 +53,9 @@
         <material>Gazebo/Orange</material>
       </xacro:if>
+      <mu1 value="0.09" />
+      <mu2 value="0.09" />
+      <kp value="10000000.0" />
+      <kd value="10000" />
+      <fdir1 value="0 0 0" />
     </gazebo>
     <link
@@ -63,5 +68,5 @@
           value="${mass}" />
         <inertia ixx="${ixx}" ixy="${ixy}" ixz="${ixz}"
-                 iyy="${iyy}" iyz="${iyz}" izz="${izz}" />
+          iyy="${iyy}" iyz="${iyz}" izz="${izz}" />
       </inertial>
       <visual>
@@ -97,9 +102,9 @@
         link="chassis" />
       <child
-        link="${part}"/>
+        link="${part}" />
       <axis
         xyz="${x_axs} 0 0" />
       <limit
-        effort="10"
+        effort="5"
         velocity="100000" />
       <dynamics
@@ -121,35 +126,35 @@
   </xacro:macro>
   <!-- base link setup -->
-  <xacro:links  part="chassis" msh="${chassis_msh}" color="white" mass="8"
-                xyz_lnk="-0.00074513 -0.11739 0.055785"
-                ixx="0.55567" ixy="-0.00039063" ixz="-0.0032652"
-                iyy="0.57391" iyz="-0.019683" izz="0.61063"/>
+  <xacro:links part="chassis" msh="${chassis_msh}" color="white" mass="8"
+    xyz_lnk="-0.00074513 -0.11739 0.055785"
+    ixx="0.55567" ixy="-0.00039063" ixz="-0.0032652"
+    iyy="0.57391" iyz="-0.019683" izz="0.61063" />
   <!-- LF_wheel setup -->
-  <xacro:links  part="LF_wheel" msh="${LF_wheel_msh}" color="orange" mass="0.49554"
-                xyz_lnk="-0.032026 -1.3878E-17 -5.5511E-17"
-                ixx="0.0018121" ixy="2.1263E-22" ixz="1.9263E-20"
-                iyy="0.00096656" iyz="5.0211E-21" izz="0.00096656"/>
-  <xacro:joints part="LF_wheel" jnt="LF_wheel_jnt" xyz_jnt="-0.27192 0.1695 -0.1241" x_axs="1"/>
-  <xacro:wheel_transmission part="LF_wheel" jnt="LF_wheel_jnt" motor="LF_wheel_motor" reduction="1"/>
+  <xacro:links part="LF_wheel" msh="${LF_wheel_msh}" color="orange" mass="0.49554"
+    xyz_lnk="-0.032026 -1.3878E-17 -5.5511E-17"
+    ixx="0.0018121" ixy="2.1263E-22" ixz="1.9263E-20"
+    iyy="0.00096656" iyz="5.0211E-21" izz="0.00096656" />
+  <xacro:joints part="LF_wheel" jnt="LF_wheel_jnt" xyz_jnt="-0.27192 0.1695 -0.1241" x_axs="1" />
+  <xacro:wheel_transmission part="LF_wheel" jnt="LF_wheel_jnt" motor="LF_wheel_motor" reduction="1" />
   <!-- LB_wheel setup -->
-  <xacro:links  part="LB_wheel" msh="${LB_wheel_msh}" color="orange" mass="0.49554"
-                xyz_lnk="-0.032026 2.7756E-17 2.7756E-17"
-                ixx="0.0018121" ixy="2.1243E-20" ixz="3.9097E-21"
-                iyy="0.00096656" iyz="9.7862E-20" izz="0.00096656"/>
-  <xacro:joints part="LB_wheel" jnt="LB_wheel_jnt" xyz_jnt="-0.27192 -0.2695 -0.1241" x_axs="1"/>
-  <xacro:wheel_transmission part="LB_wheel" jnt="LB_wheel_jnt" motor="LB_wheel_motor" reduction="1"/>
+  <xacro:links part="LB_wheel" msh="${LB_wheel_msh}" color="orange" mass="0.49554"
+    xyz_lnk="-0.032026 2.7756E-17 2.7756E-17"
+    ixx="0.0018121" ixy="2.1243E-20" ixz="3.9097E-21"
+    iyy="0.00096656" iyz="9.7862E-20" izz="0.00096656" />
+  <xacro:joints part="LB_wheel" jnt="LB_wheel_jnt" xyz_jnt="-0.27192 -0.2695 -0.1241" x_axs="1" />
+  <xacro:wheel_transmission part="LB_wheel" jnt="LB_wheel_jnt" motor="LB_wheel_motor" reduction="1" />
   <!-- RF_wheel setup -->
   <xacro:links part="RF_wheel" msh="${RF_wheel_msh}" color="orange" mass="0.49554"
-                xyz_lnk="0.032026 6.9389E-17 0"
-                ixx="0.0018121" ixy="1.1755E-35" ixz="2.5636E-20"
-                iyy="0.00096656" iyz="3.8844E-35" izz="0.00096656"/>
-  <xacro:joints part="RF_wheel" jnt="RF_wheel_jnt" xyz_jnt="0.27208 0.1695 -0.1241" x_axs="-1"/>
-  <xacro:wheel_transmission part="RF_wheel" jnt="RF_wheel_jnt" motor="RF_wheel_motor" reduction="1"/>
+    xyz_lnk="0.032026 6.9389E-17 0"
+    ixx="0.0018121" ixy="1.1755E-35" ixz="2.5636E-20"
+    iyy="0.00096656" iyz="3.8844E-35" izz="0.00096656" />
+  <xacro:joints part="RF_wheel" jnt="RF_wheel_jnt" xyz_jnt="0.27208 0.1695 -0.1241" x_axs="-1" />
+  <xacro:wheel_transmission part="RF_wheel" jnt="RF_wheel_jnt" motor="RF_wheel_motor" reduction="1" />
   <!-- RB_wheel setup -->
-  <xacro:links  part="RB_wheel" msh="${RB_wheel_msh}" color="orange" mass="0.49554"
-                xyz_lnk="0.032026 6.9389E-17 0"
-                ixx="0.0018121" ixy="3.3987E-36" ixz="1.3212E-20"
-                iyy="0.00096656" iyz="-4.9432E-36" izz="0.00096656"/>
-  <xacro:joints part="RB_wheel" jnt="RB_wheel_jnt" xyz_jnt="0.27208 -0.2695 -0.1241" x_axs="-1"/>
-  <xacro:wheel_transmission part="RB_wheel" jnt="RB_wheel_jnt" motor="RB_wheel_motor" reduction="1"/>
+  <xacro:links part="RB_wheel" msh="${RB_wheel_msh}" color="orange" mass="0.49554"
+    xyz_lnk="0.032026 6.9389E-17 0"
+    ixx="0.0018121" ixy="3.3987E-36" ixz="1.3212E-20"
+    iyy="0.00096656" iyz="-4.9432E-36" izz="0.00096656" />
+  <xacro:joints part="RB_wheel" jnt="RB_wheel_jnt" xyz_jnt="0.27208 -0.2695 -0.1241" x_axs="-1" />
+  <xacro:wheel_transmission part="RB_wheel" jnt="RB_wheel_jnt" motor="RB_wheel_motor" reduction="1" />
 </robot>
