Commit message: Change project name

File: asado_description/urdf/asado.xacro (robot description, xacro)
@@ -2,13 +2,13 @@
 <robot xmlns:xacro="http://www.ros.org/wiki/xacro" name="asado">
   <!-- Import Rviz colors -->
-  <xacro:include filename="$(find asado_simulation)/urdf/materials.xacro" />
-  <xacro:include filename="$(find asado_simulation)/urdf/asado.gazebo" />
+  <xacro:include filename="$(find asado_description)/urdf/materials.xacro" />
+  <xacro:include filename="$(find asado_description)/urdf/asado.gazebo" />
   <!-- Define the model path -->
-  <xacro:property name="chassis_msh" value="package://asado_simulation/meshes/chassis.STL" />
-  <xacro:property name="LF_wheel_msh" value="package://asado_simulation/meshes/LF_wheel.STL" />
-  <xacro:property name="LB_wheel_msh" value="package://asado_simulation/meshes/LB_wheel.STL" />
-  <xacro:property name="RF_wheel_msh" value="package://asado_simulation/meshes/RF_wheel.STL" />
-  <xacro:property name="RB_wheel_msh" value="package://asado_simulation/meshes/RB_wheel.STL" />
-  <xacro:property name="hokuyo_msh" value="package://asado_simulation/meshes/hokuyo.dae" />
+  <xacro:property name="chassis_msh" value="package://asado_description/meshes/chassis.STL" />
+  <xacro:property name="LF_wheel_msh" value="package://asado_description/meshes/LF_wheel.STL" />
+  <xacro:property name="LB_wheel_msh" value="package://asado_description/meshes/LB_wheel.STL" />
+  <xacro:property name="RF_wheel_msh" value="package://asado_description/meshes/RF_wheel.STL" />
+  <xacro:property name="RB_wheel_msh" value="package://asado_description/meshes/RB_wheel.STL" />
+  <xacro:property name="hokuyo_msh" value="package://asado_description/meshes/hokuyo.dae" />
   <!-- Dummy link and joint used for baselink footprint -->
   <link name="base_link"></link>

Commit message: Rename base_link to footprint

File: asado_description/urdf/asado.xacro (robot description, xacro)
@@ -11,8 +11,8 @@
   <xacro:property name="RB_wheel_msh" value="package://asado_description/meshes/RB_wheel.STL" />
   <xacro:property name="hokuyo_msh" value="package://asado_description/meshes/hokuyo.dae" />
-  <!-- Dummy link and joint used for baselink footprint -->
-  <link name="base_link"></link>
+  <!-- Dummy link and joint used for footprint -->
+  <link name="footprint"></link>
   <joint name="base_jnt" type="fixed">
-    <parent link="base_link" />
+    <parent link="footprint" />
     <child link="chassis" />
   </joint>

Commit message: Update model params

File: asado_description/urdf/asado.xacro (robot description, xacro)
@@ -11,4 +11,6 @@
   <xacro:property name="RB_wheel_msh" value="package://asado_description/meshes/RB_wheel.STL" />
   <xacro:property name="hokuyo_msh" value="package://asado_description/meshes/hokuyo.dae" />
+  <!-- Define the model property -->
+  <xacro:property name="wheel_mass" value="0.8" />
   <!-- Dummy link and joint used for footprint -->
   <link name="footprint"></link>
@@ -53,6 +55,6 @@
         <material>Gazebo/Orange</material>
       </xacro:if>
-      <mu1 value="0.09" />
-      <mu2 value="0.09" />
+      <mu1 value="1.5" />
+      <mu2 value="1.5" />
       <kp value="10000000.0" />
       <kd value="10000" />
@@ -131,5 +133,5 @@
     iyy="0.57391" iyz="-0.019683" izz="0.61063" />
   <!-- LF_wheel setup -->
-  <xacro:links part="LF_wheel" msh="${LF_wheel_msh}" color="orange" mass="0.49554"
+  <xacro:links part="LF_wheel" msh="${LF_wheel_msh}" color="orange" mass="${wheel_mass}"
     xyz_lnk="-0.032026 -1.3878E-17 -5.5511E-17"
     ixx="0.0018121" ixy="2.1263E-22" ixz="1.9263E-20"
@@ -138,5 +140,5 @@
   <xacro:wheel_transmission part="LF_wheel" jnt="LF_wheel_jnt" motor="LF_wheel_motor" reduction="1" />
   <!-- LB_wheel setup -->
-  <xacro:links part="LB_wheel" msh="${LB_wheel_msh}" color="orange" mass="0.49554"
+  <xacro:links part="LB_wheel" msh="${LB_wheel_msh}" color="orange" mass="${wheel_mass}"
     xyz_lnk="-0.032026 2.7756E-17 2.7756E-17"
     ixx="0.0018121" ixy="2.1243E-20" ixz="3.9097E-21"
@@ -145,5 +147,5 @@
   <xacro:wheel_transmission part="LB_wheel" jnt="LB_wheel_jnt" motor="LB_wheel_motor" reduction="1" />
   <!-- RF_wheel setup -->
-  <xacro:links part="RF_wheel" msh="${RF_wheel_msh}" color="orange" mass="0.49554"
+  <xacro:links part="RF_wheel" msh="${RF_wheel_msh}" color="orange" mass="${wheel_mass}"
     xyz_lnk="0.032026 6.9389E-17 0"
     ixx="0.0018121" ixy="1.1755E-35" ixz="2.5636E-20"
@@ -152,5 +154,5 @@
   <xacro:wheel_transmission part="RF_wheel" jnt="RF_wheel_jnt" motor="RF_wheel_motor" reduction="1" />
   <!-- RB_wheel setup -->
-  <xacro:links part="RB_wheel" msh="${RB_wheel_msh}" color="orange" mass="0.49554"
+  <xacro:links part="RB_wheel" msh="${RB_wheel_msh}" color="orange" mass="${wheel_mass}"
     xyz_lnk="0.032026 6.9389E-17 0"
     ixx="0.0018121" ixy="3.3987E-36" ixz="1.3212E-20"

Commit message: Change lidar position

File: asado_description/urdf/asado.xacro (robot description, xacro)
@@ -22,5 +22,5 @@
   <joint name="hokuyo_joint" type="fixed">
     <axis xyz="0 1 0" />
-    <origin xyz="0 0 0.05" rpy="0 0 0" />
+    <origin xyz="0 0.25 0.05" rpy="0 0 0" />
     <parent link="chassis" />
     <child link="hokuyo_link" />

Commit message: Tweak lidar position

File: asado_description/urdf/asado.xacro (robot description, xacro)
@@ -22,5 +22,5 @@
   <joint name="hokuyo_joint" type="fixed">
     <axis xyz="0 1 0" />
-    <origin xyz="0 0.25 0.05" rpy="0 0 0" />
+    <origin xyz="0 0 0.05" rpy="0 0 0" />
     <parent link="chassis" />
     <child link="hokuyo_link" />

Commit message: Change directory

File: asado_description/urdf/asado.xacro (robot description, xacro)
@@ -1,162 +1,33 @@
 <?xml version="1.0" encoding="utf-8"?>
 <robot xmlns:xacro="http://www.ros.org/wiki/xacro" name="asado">
-  <!-- Import Rviz colors -->
-  <xacro:include filename="$(find asado_description)/urdf/materials.xacro" />
-  <xacro:include filename="$(find asado_description)/urdf/asado.gazebo" />
-  <!-- Define the model path -->
-  <xacro:property name="chassis_msh" value="package://asado_description/meshes/chassis.STL" />
-  <xacro:property name="LF_wheel_msh" value="package://asado_description/meshes/LF_wheel.STL" />
-  <xacro:property name="LB_wheel_msh" value="package://asado_description/meshes/LB_wheel.STL" />
-  <xacro:property name="RF_wheel_msh" value="package://asado_description/meshes/RF_wheel.STL" />
-  <xacro:property name="RB_wheel_msh" value="package://asado_description/meshes/RB_wheel.STL" />
-  <xacro:property name="hokuyo_msh" value="package://asado_description/meshes/hokuyo.dae" />
-  <!-- Define the model property -->
-  <xacro:property name="wheel_mass" value="0.8" />
-  <!-- Dummy link and joint used for footprint -->
-  <link name="footprint"></link>
-  <joint name="base_jnt" type="fixed">
-    <parent link="footprint" />
-    <child link="chassis" />
-  </joint>
-  <!-- Lidar Joint -->
-  <joint name="hokuyo_joint" type="fixed">
-    <axis xyz="0 1 0" />
-    <origin xyz="0 0 0.05" rpy="0 0 0" />
-    <parent link="chassis" />
-    <child link="hokuyo_link" />
-  </joint>
-  <!-- Lidar Link -->
-  <link name="hokuyo_link">
-    <collision>
-      <origin xyz="0 0 0" rpy="0 0 0" />
-      <geometry>
-        <mesh filename="${hokuyo_msh}" />
-      </geometry>
-    </collision>
-    <visual>
-      <origin xyz="0 0 0" rpy="0 0 0" />
-      <geometry>
-        <mesh filename="${hokuyo_msh}" />
-      </geometry>
-    </visual>
-    <inertial>
-      <mass value="1E-5" />
-      <origin xyz="0 0 0" rpy="0 0 0" />
-      <inertia ixx="1E-6" ixy="0" ixz="0" iyy="1E-6" iyz="0" izz="1E-6" />
-    </inertial>
-  </link>
-  <!-- Macro for Links -->
-  <xacro:macro name="links" params="part msh color mass xyz_lnk ixx ixy ixz iyy iyz izz">
-    <gazebo reference="${part}">
-      <xacro:if value="${color == 'white'}">
-        <material>Gazebo/White</material>
-      </xacro:if>
-      <xacro:if value="${color == 'orange'}">
-        <material>Gazebo/Orange</material>
-      </xacro:if>
-      <mu1 value="1.5" />
-      <mu2 value="1.5" />
-      <kp value="10000000.0" />
-      <kd value="10000" />
-      <fdir1 value="0 0 0" />
-    </gazebo>
-    <link
-      name="${part}">
-      <inertial>
-        <origin
-          xyz="${xyz_lnk}"
-          rpy="0 0 0" />
-        <mass
-          value="${mass}" />
-        <inertia ixx="${ixx}" ixy="${ixy}" ixz="${ixz}"
-          iyy="${iyy}" iyz="${iyz}" izz="${izz}" />
-      </inertial>
-      <visual>
-        <origin
-          xyz="0 0 0"
-          rpy="0 0 0" />
-        <geometry>
-          <mesh
-            filename="${msh}" />
-        </geometry>
-        <material name="${color}" />
-      </visual>
-      <collision>
-        <origin
-          xyz="0 0 0"
-          rpy="0 0 0" />
-        <geometry>
-          <mesh
-            filename="${msh}" />
-        </geometry>
-      </collision>
-    </link>
-  </xacro:macro>
-  <!-- Macro for Joints -->
-  <xacro:macro name="joints" params="part jnt xyz_jnt x_axs">
-    <joint
-      name="${jnt}"
-      type="continuous">
-      <origin
-        xyz="${xyz_jnt}"
-        rpy="0 0 0" />
-      <parent
-        link="chassis" />
-      <child
-        link="${part}" />
-      <axis
-        xyz="${x_axs} 0 0" />
-      <limit
-        effort="5"
-        velocity="100000" />
-      <dynamics
-        damping="0.8" />
-    </joint>
-  </xacro:macro>
-  <!-- Macro for Wheel transmissions -->
-  <xacro:macro name="wheel_transmission" params="part jnt motor reduction">
-    <transmission name="${part}">
-      <type>transmission_interface/SimpleTransmission</type>
-      <joint name="${jnt}">
-        <hardwareInterface>hardware_interface/VelocityJointInterface</hardwareInterface>
-      </joint>
-      <actuator name="${motor}">
-        <hardwareInterface>hardware_interface/VelocityJointInterface</hardwareInterface>
-        <mechanicalReduction value="${reduction}" />
-      </actuator>
-    </transmission>
-  </xacro:macro>
-  <!-- base link setup -->
-  <xacro:links part="chassis" msh="${chassis_msh}" color="white" mass="8"
-    xyz_lnk="-0.00074513 -0.11739 0.055785"
-    ixx="0.55567" ixy="-0.00039063" ixz="-0.0032652"
-    iyy="0.57391" iyz="-0.019683" izz="0.61063" />
-  <!-- LF_wheel setup -->
-  <xacro:links part="LF_wheel" msh="${LF_wheel_msh}" color="orange" mass="${wheel_mass}"
-    xyz_lnk="-0.032026 -1.3878E-17 -5.5511E-17"
-    ixx="0.0018121" ixy="2.1263E-22" ixz="1.9263E-20"
-    iyy="0.00096656" iyz="5.0211E-21" izz="0.00096656" />
-  <xacro:joints part="LF_wheel" jnt="LF_wheel_jnt" xyz_jnt="-0.27192 0.1695 -0.1241" x_axs="-1" />
-  <xacro:wheel_transmission part="LF_wheel" jnt="LF_wheel_jnt" motor="LF_wheel_motor" reduction="1" />
-  <!-- LB_wheel setup -->
-  <xacro:links part="LB_wheel" msh="${LB_wheel_msh}" color="orange" mass="${wheel_mass}"
-    xyz_lnk="-0.032026 2.7756E-17 2.7756E-17"
-    ixx="0.0018121" ixy="2.1243E-20" ixz="3.9097E-21"
-    iyy="0.00096656" iyz="9.7862E-20" izz="0.00096656" />
-  <xacro:joints part="LB_wheel" jnt="LB_wheel_jnt" xyz_jnt="-0.27192 -0.2695 -0.1241" x_axs="-1" />
-  <xacro:wheel_transmission part="LB_wheel" jnt="LB_wheel_jnt" motor="LB_wheel_motor" reduction="1" />
-  <!-- RF_wheel setup -->
-  <xacro:links part="RF_wheel" msh="${RF_wheel_msh}" color="orange" mass="${wheel_mass}"
-    xyz_lnk="0.032026 6.9389E-17 0"
-    ixx="0.0018121" ixy="1.1755E-35" ixz="2.5636E-20"
-    iyy="0.00096656" iyz="3.8844E-35" izz="0.00096656" />
-  <xacro:joints part="RF_wheel" jnt="RF_wheel_jnt" xyz_jnt="0.27208 0.1695 -0.1241" x_axs="-1" />
-  <xacro:wheel_transmission part="RF_wheel" jnt="RF_wheel_jnt" motor="RF_wheel_motor" reduction="1" />
-  <!-- RB_wheel setup -->
-  <xacro:links part="RB_wheel" msh="${RB_wheel_msh}" color="orange" mass="${wheel_mass}"
-    xyz_lnk="0.032026 6.9389E-17 0"
-    ixx="0.0018121" ixy="3.3987E-36" ixz="1.3212E-20"
-    iyy="0.00096656" iyz="-4.9432E-36" izz="0.00096656" />
-  <xacro:joints part="RB_wheel" jnt="RB_wheel_jnt" xyz_jnt="0.27208 -0.2695 -0.1241" x_axs="-1" />
-  <xacro:wheel_transmission part="RB_wheel" jnt="RB_wheel_jnt" motor="RB_wheel_motor" reduction="1" />
+  <!-- Import components -->
+  <xacro:include filename="$(find asado_description)/urdf/include/materials.xacro" />
+  <xacro:include filename="$(find asado_description)/urdf/include/plugin.xacro" />
+  <xacro:include filename="$(find asado_description)/urdf/include/chassis.xacro" />
+  <xacro:include filename="$(find asado_description)/urdf/include/wheel.xacro"/>
+  <xacro:include filename="$(find asado_description)/urdf/include/sensor.xacro"/>
+  <xacro:property name="chassis_yaml" value="$(find asado_description)/config/chassis.yaml" />
+  <xacro:property name="chassis_props" value="${xacro.load_yaml(chassis_yaml)}"/>
+  <xacro:property name="LF_wheel_yaml" value="$(find asado_description)/config/wheels/LF_wheel.yaml" />
+  <xacro:property name="LF_wheel_props" value="${xacro.load_yaml(LF_wheel_yaml)}"/>
+  <xacro:property name="LB_wheel_yaml" value="$(find asado_description)/config/wheels/LB_wheel.yaml" />
+  <xacro:property name="LB_wheel_props" value="${xacro.load_yaml(LB_wheel_yaml)}"/>
+  <xacro:property name="RF_wheel_yaml" value="$(find asado_description)/config/wheels/RF_wheel.yaml" />
+  <xacro:property name="RF_wheel_props" value="${xacro.load_yaml(RF_wheel_yaml)}"/>
+  <xacro:property name="RB_wheel_yaml" value="$(find asado_description)/config/wheels/RB_wheel.yaml" />
+  <xacro:property name="RB_wheel_props" value="${xacro.load_yaml(RB_wheel_yaml)}"/>
+  <xacro:property name="sensor_yaml" value="$(find asado_description)/config/sensor.yaml" />
+  <xacro:property name="sensor_props" value="${xacro.load_yaml(sensor_yaml)}"/>
+  <!-- Chassis -->
+  <xacro:chassis chassis_props="${chassis_props}" />
+  <!-- Wheels -->
+  <xacro:wheel wheel_props="${LF_wheel_props}" />
+  <xacro:wheel wheel_props="${LB_wheel_props}" />
+  <xacro:wheel wheel_props="${RF_wheel_props}" />
+  <xacro:wheel wheel_props="${RB_wheel_props}" />
+  <!-- Sensors -->
+  <xacro:lidar lidar_props="${sensor_props}" />
+  <!-- Plugin -->
+  <xacro:gazebo_ros_control />
+  <xacro:gazebo_ros_control />
 </robot>

Commit message: Change lidar position

File: asado_description/urdf/asado.xacro (robot description, xacro)
@@ -22,5 +22,5 @@
   <joint name="hokuyo_joint" type="fixed">
     <axis xyz="0 1 0" />
-    <origin xyz="0 0 0.05" rpy="0 0 0" />
+    <origin xyz="0 0.3 0.05" rpy="0 0 0" />
     <parent link="chassis" />
     <child link="hokuyo_link" />
@@ -55,6 +55,6 @@
         <material>Gazebo/Orange</material>
       </xacro:if>
-      <mu1 value="1.5" />
-      <mu2 value="1.5" />
+      <mu1 value="100" />
+      <mu2 value="100" />
       <kp value="10000000.0" />
       <kd value="10000" />

Commit message: Reorganize files

File: asado_description/urdf/asado.xacro (robot description, xacro)
@@ -30,4 +30,4 @@
   <!-- Plugin -->
   <xacro:gazebo_ros_control />
-  <xacro:gazebo_ros_control />
+  <xacro:skid_steer_drive_controller />
 </robot>

File: asado_description/urdf/include/plugin.xacro (robot description, xacro)
@@ -11,5 +11,5 @@
 	</xacro:macro>
 	<!-- skid_steer_drive_controller -->
-	<xacro:macro name="gazebo_ros_control" params="">
+	<xacro:macro name="skid_steer_drive_controller" params="">
 		<gazebo>
 			<plugin name="skid_steer_drive_controller" filename="libgazebo_ros_skid_steer_drive.so">
