Commit message: Change the direction of robot face

File: asado_description/urdf/include/chassis.xacro (robot description, xacro)
@@ -7,4 +7,6 @@
 			<parent link="footprint" />
 			<child link="chassis" />
+      <!-- Rotate 90 degrees along z-axis -->
+      <origin rpy="0 0 -1.5708" />
 		</joint>
 		<!-- Link -->
