Commit message: Update move base params

File: asado_description/urdf/include/plugin.xacro (robot description, xacro)
@@ -23,6 +23,6 @@
 				<wheelDiameter>1.54</wheelDiameter>
 				<robotBaseFrame>footprint</robotBaseFrame>
-				<MaxForce>100.0</MaxForce>
-				<torque>200</torque>
+				<MaxForce>1000.0</MaxForce>
+				<torque>1000</torque>
 				<commandTopic>cmd_vel</commandTopic>
 				<odometryTopic>odom</odometryTopic>

File: asado_description/urdf/include/wheel.xacro (robot description, xacro)
@@ -16,8 +16,8 @@
         <material>Gazebo/Green</material>
       </xacro:if>
-      <mu1 value="${wheel_props['link']['mu1']}" />
-      <mu2 value="${wheel_props['link']['mu2']}" />
-      <kp value="${wheel_props['link']['kp']}" />
-      <kd value="${wheel_props['link']['kd']}" />
+      <mu1 value="1" />
+      <mu2 value="1" />
+      <kp value="1e+13" />
+      <kd value="1" />
       <fdir1 value="0 0 0" />
     </gazebo>
@@ -49,6 +49,6 @@
       <child link="${wheel_props['joint']['child_link']}" />
       <axis xyz="${wheel_props['joint']['x_axs']} 0 0" />
-      <limit effort="${wheel_props['joint']['effort']}" velocity="${wheel_props['joint']['velocity']}" />
-      <dynamics damping="${wheel_props['joint']['damping']}" />
+      <limit effort="1000" velocity="1000000" />
+      <dynamics damping="0" />
     </joint>
     <!-- Macro for Wheel transmission -->
