Commit message: Update navigation stack params

File: asado_description/urdf/include/wheel.xacro (robot description, xacro)
@@ -16,8 +16,8 @@
         <material>Gazebo/Green</material>
       </xacro:if>
-      <mu1 value="1" />
-      <mu2 value="1" />
-      <kp value="1e+13" />
-      <kd value="1" />
+      <mu1 value="200" />
+      <mu2 value="200" />
+      <kp value="10000000.0" />
+      <kd value="1.0" />
       <fdir1 value="0 0 0" />
     </gazebo>
@@ -49,6 +49,6 @@
       <child link="${wheel_props['joint']['child_link']}" />
       <axis xyz="${wheel_props['joint']['x_axs']} 0 0" />
-      <limit effort="1000" velocity="1000000" />
-      <dynamics damping="0" />
+      <!-- <limit effort="1000" velocity="1000000" /> -->
+      <!-- <dynamics damping="0.01" fraction="0.0"/> -->
     </joint>
     <!-- Macro for Wheel transmission -->
