Commit message: Attempt to fix low cmd_vel published by move_base

File: pollo_description/urdf/include/wheel.xacro (robot description, xacro)
@@ -20,5 +20,5 @@
       <kp value="10000000.0" />
       <kd value="1.0" />
-      <fdir1 value="0 0 0" />
+      <minDepth>0.01</minDepth>
     </gazebo>
     <link name="${wheel_props['link']['name']}">
@@ -49,6 +49,4 @@
       <child link="${wheel_props['joint']['child_link']}" />
       <axis xyz="${wheel_props['joint']['x_axs']} 0 0" />
-      <!-- <limit effort="1000" velocity="1000000" /> -->
-      <!-- <dynamics damping="0.01" fraction="0.0"/> -->
     </joint>
     <!-- Macro for Wheel transmission -->
