Commit message: Update link name

File: pollo_description/urdf/include/sensor.xacro (robot description, xacro)
@@ -3,16 +3,16 @@
   <xacro:macro name="lidar" params="lidar_props">
     <!-- Joint -->
-    <joint name="hokuyo_joint" type="fixed">
+    <joint name="laser_joint" type="fixed">
       <axis xyz="0 1 0" />
-      <origin xyz="${sensor_props['lidar']['hokuyo']['x']} ${sensor_props['lidar']['hokuyo']['y']} ${sensor_props['lidar']['hokuyo']['z']}" rpy="0 0 0" />
+      <origin xyz="${sensor_props['lidar']['laser']['x']} ${sensor_props['lidar']['laser']['y']} ${sensor_props['lidar']['laser']['z']}" rpy="0 0 0" />
       <parent link="chassis" />
-      <child link="hokuyo_link" />
+      <child link="laser_link" />
     </joint>
     <!-- Link -->
-    <link name="hokuyo_link">
+    <link name="laser_link">
       <collision>
         <origin xyz="0 0 0" rpy="0 0 0" />
         <geometry>
-          <mesh filename="${sensor_props['lidar']['hokuyo']['msh']}" />
+          <mesh filename="${sensor_props['lidar']['laser']['msh']}" />
         </geometry>
       </collision>
@@ -20,5 +20,5 @@
         <origin xyz="0 0 0" rpy="0 0 0" />
         <geometry>
-          <mesh filename="${sensor_props['lidar']['hokuyo']['msh']}" />
+          <mesh filename="${sensor_props['lidar']['laser']['msh']}" />
         </geometry>
       </visual>
@@ -29,8 +29,8 @@
       </inertial>
     </link>
-    <gazebo reference="hokuyo_link">
+    <gazebo reference="laser_link">
       <sensor type="ray" name="laser_sensor">
         <pose>0 0 0 0 0 0</pose>
-        <visualize>${sensor_props['lidar']['hokuyo']['visualize']}</visualize>
+        <visualize>${sensor_props['lidar']['laser']['visualize']}</visualize>
         <update_rate>40</update_rate>
         <ray>
@@ -39,16 +39,16 @@
               <samples>720</samples>
               <resolution>1</resolution>
-              <min_angle>${sensor_props['lidar']['hokuyo']['min_angle']}</min_angle>
-              <max_angle>${sensor_props['lidar']['hokuyo']['max_angle']}</max_angle>
+              <min_angle>${sensor_props['lidar']['laser']['min_angle']}</min_angle>
+              <max_angle>${sensor_props['lidar']['laser']['max_angle']}</max_angle>
             </horizontal>
           </scan>
           <range>
-            <min>${sensor_props['lidar']['hokuyo']['min_range']}</min>
-            <max>${sensor_props['lidar']['hokuyo']['max_range']}</max>
+            <min>${sensor_props['lidar']['laser']['min_range']}</min>
+            <max>${sensor_props['lidar']['laser']['max_range']}</max>
             <resolution>0.01</resolution>
           </range>
           <noise>
             <type>gaussian</type>
-            <!-- Noise parameters based on published spec for Hokuyo laser
+            <!-- Noise parameters based on published spec for laser laser
                 achieving "+-30mm" accuracy at range < 10m.  A mean of 0.0m and
                 stddev of 0.01m will put 99.7% of samples within 0.03m of the true
@@ -58,7 +58,7 @@
           </noise>
         </ray>
-        <plugin name="gazebo_ros_head_hokuyo_controller" filename="libgazebo_ros_laser.so">
+        <plugin name="gazebo_ros_head_laser_controller" filename="libgazebo_ros_laser.so">
           <topicName>/pollo/laser/scan</topicName>
-          <frameName>hokuyo_link</frameName>
+          <frameName>laser_link</frameName>
         </plugin>
       </sensor>
